File: _autosave-Pulse generator daughter board.kicad_pcb (KiCad board)
At the start: 2 copper layers, 31 parts, among them U1 MAX31855KASA, U3 TC4427, U4 TC4427

Commit message: Progress 2 on schematic and PCB
Parts:
- added J15: ~, Connector_PinHeader_2.54mm:PinHeader_2x08_P2.54mm_Vertical, F.Cu at (195.0, 47.8)
- added J16: ~, Connector_PinHeader_2.54mm:PinHeader_2x15_P2.54mm_Vertical, F.Cu at (194.5, 90.1)
- added J17: ~, Connector_PinHeader_2.54mm:PinHeader_2x10_P2.54mm_Vertical, F.Cu at (237.5, 47.6)
- added J18: ~, Connector_PinHeader_2.54mm:PinHeader_2x17_P2.54mm_Vertical, F.Cu at (239.5, 88.4)
- moved U4 9.00 mm to (124.3, 110.2)
- moved D1 9.00 mm to (121.0, 159.0)
- moved R22 9.00 mm to (116.5, 133.0)
- moved R23 9.00 mm to (123.5, 133.0)
- moved R24 9.00 mm to (116.5, 146.0)
- moved R25 9.00 mm to (123.5, 145.9)
Other:
- copper layers 2 -> 4

Commit message: Progress on PCB 29.11.2024
Parts:
- removed R26: 10k, Resistor_SMD:R_0805_2012Metric_Pad1.20x1.40mm_HandSolder
- added C1: C, Capacitor_SMD:C_0805_2012Metric_Pad1.18x1.45mm_HandSolder, F.Cu at (107.5, 87.5)
- added C10: C, Capacitor_SMD:C_0805_2012Metric_Pad1.18x1.45mm_HandSolder, F.Cu at (44.7, 105.5)
- added C11: C, Capacitor_SMD:C_0805_2012Metric_Pad1.18x1.45mm_HandSolder, F.Cu at (44.7, 108.5)
- added C12: 100nF, Capacitor_SMD:C_0805_2012Metric_Pad1.18x1.45mm_HandSolder, F.Cu at (106.0, 120.0)
- added C13: 100nF, Capacitor_SMD:C_0805_2012Metric_Pad1.18x1.45mm_HandSolder, F.Cu at (107.5, 137.0)
- added C14: 100nF, Capacitor_SMD:C_0805_2012Metric_Pad1.18x1.45mm_HandSolder, F.Cu at (78.0, 115.0)
- added C15: 100nF, Capacitor_SMD:C_0805_2012Metric_Pad1.18x1.45mm_HandSolder, F.Cu at (93.5, 115.0)
- added C2: C, Capacitor_SMD:C_0805_2012Metric_Pad1.18x1.45mm_HandSolder, F.Cu at (80.5, 99.0)
- added C3: 10nF, Capacitor_SMD:C_0805_2012Metric_Pad1.18x1.45mm_HandSolder, F.Cu at (118.0, 135.0)
- added C4: C, Capacitor_SMD:C_0805_2012Metric_Pad1.18x1.45mm_HandSolder, F.Cu at (109.5, 113.0)
- added C5: 100nF, Capacitor_SMD:C_0805_2012Metric_Pad1.18x1.45mm_HandSolder, F.Cu at (118.0, 131.5)
- added C6: C, Capacitor_SMD:C_0805_2012Metric_Pad1.18x1.45mm_HandSolder, F.Cu at (109.5, 115.5)
- added C7: C, Capacitor_SMD:C_0805_2012Metric_Pad1.18x1.45mm_HandSolder, F.Cu at (39.8, 108.5)
- added C8: C, Capacitor_SMD:C_0805_2012Metric_Pad1.18x1.45mm_HandSolder, F.Cu at (44.7, 99.5)
- added C9: C, Capacitor_SMD:C_0805_2012Metric_Pad1.18x1.45mm_HandSolder, F.Cu at (94.0, 98.5)
- added J1: Vin1, Connector_Wire:SolderWire-0.5sqmm_1x01_D0.9mm_OD2.1mm, F.Cu at (77.0, 46.5)
- added J10: Vin2_GND, Connector_Wire:SolderWire-0.5sqmm_1x01_D0.9mm_OD2.1mm, F.Cu at (109.0, 51.5)
- added J15: CH1 output, Connector_Wire:SolderWire-0.5sqmm_1x01_D0.9mm_OD2.1mm, F.Cu at (66.5, 135.0)
- added J16: GND, Connector_Wire:SolderWire-0.5sqmm_1x01_D0.9mm_OD2.1mm, F.Cu at (66.5, 140.0)
- added J17: CH2 output, Connector_Wire:SolderWire-0.5sqmm_1x01_D0.9mm_OD2.1mm, F.Cu at (85.0, 135.0)
- added J18: GND, Connector_Wire:SolderWire-0.5sqmm_1x01_D0.9mm_OD2.1mm, F.Cu at (85.0, 140.0)
- added J2: Vin1_GND, Connector_Wire:SolderWire-0.5sqmm_1x01_D0.9mm_OD2.1mm, F.Cu at (77.0, 51.5)
- added J7: T+, Connector_Wire:SolderWire-0.5sqmm_1x01_D0.9mm_OD2.1mm, F.Cu at (120.0, 139.5)
- added J8: T-, Connector_Wire:SolderWire-0.5sqmm_1x01_D0.9mm_OD2.1mm, F.Cu at (114.0, 139.5)
- added J9: Vin2, Connector_Wire:SolderWire-0.5sqmm_1x01_D0.9mm_OD2.1mm, F.Cu at (109.0, 46.5)
- added U1: RYK-053.3SH, Rafal:RYK-053.3SH, F.Cu at (109.8, 93.5)
- added U3: ADUM1402, Package_SO:SOIC-16W_7.5x10.3mm_P1.27mm, F.Cu at (109.0, 128.0)
- J11: renamed from J15; value ~ -> CN8
- J12: renamed from J16; value ~ -> CN9
- J13: renamed from J17; value ~ -> CN7
- J14: renamed from J18; value ~ -> CN10
- moved J12 127.3 mm to (67.5, 82.1)
- moved J11 127.0 mm to (68.0, 47.8)
- moved J14 123.0 mm to (117.0, 77.2)
- moved J13 120.5 mm to (117.0, 47.3)
- moved R16 84.6 mm to (83.5, 115.0), turned to 180 degrees
- moved R17 71.1 mm to (99.0, 115.0), turned to 180 degrees
- moved D1 64.0 mm to (85.5, 47.5)
- moved R14 58.1 mm to (93.4, 71.5)
- moved R15 58.1 mm to (93.4, 74.4)
- moved D7 49.2 mm to (66.5, 126.5), turned to 90 degrees
- moved D8 48.5 mm to (85.0, 126.5), turned to 90 degrees
- moved D6 47.6 mm to (100.5, 47.5)
- moved U2 38.8 mm to (119.0, 125.5), turned to 90 degrees
- moved R22 38.6 mm to (73.0, 126.0), turned to 90 degrees
- moved R18 33.1 mm to (73.0, 135.9), turned to 90 degrees
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- renumbered D6 to D1, D8 to D6, D1 to D8, R20 to R19, R22 to R20, R23 to R21, R19 to R22, R21 to R23, U1 to U2, U3 to U4, U4 to U5
Connections:
- J11 pad 9: unconnected-(J15-Pin_9-Pad9) -> /+5V
- J12 pad 19: unconnected-(J16-Pin_19-Pad19) -> /ADC2
- J12 pad 3: unconnected-(J16-Pin_3-Pad3) -> /ADC1
- J13 pad 10: unconnected-(J17-Pin_10-Pad10) -> /PWM1 _CH1
- J13 pad 15: unconnected-(J17-Pin_15-Pad15) -> Net-(J13-Pin_15)
- J13 pad 19: unconnected-(J17-Pin_19-Pad19) -> Net-(J13-Pin_19)
- J13 pad 2: unconnected-(J17-Pin_2-Pad2) -> Net-(J13-Pin_2)
- J14 pad 29: unconnected-(J18-Pin_29-Pad29) -> /PWM1 _CH2
- R11 pad 2: unconnected-(R11-Pad2) -> GND
- R12 pad 2: Net-(J11-Pin_1) -> /ADC1
- R13 pad 2: Net-(J13-Pin_1) -> /ADC2
- R14 pad 2: Net-(J19-Pin_1) -> /PWM1 _CH1
- R15 pad 2: Net-(J20-Pin_1) -> /PWM1 _CH2
- R9 pad 2: unconnected-(R9-Pad2) -> GND
- U2 pad 4: +3V3_TC -> Net-(U1-+Vout)
- U4 pad 2: Net-(J19-Pin_1) -> /PWM1 _CH1
- U5 pad 2: Net-(J20-Pin_1) -> /PWM1 _CH2
Routing:
- net GND: track 0.00 -> 2.20 mm, vias 0 -> 1
- added copper zone on In1.Cu, net GND
- added copper zone on In2.Cu, net GND
Other:
- board outline added: 60 x 100 mm
- board text added: "60x80"
