File: _autosave-Pulse generator daughter board.kicad_sch (KiCad schematic)
At the start: 71 parts, among them J1 Vin1, J10 Vin2_GND, J11 CN8, J12 CN9, J13 CN7, J14 CN10, J15 CH1 output, J16 GND, J17 CH2 output, J18 GND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

Commit message: Connector position locked + some more progress
Parts:
- added U6: MAX31856, Package_SO:TSSOP-14_4.4x5mm_P0.65mm, symbol Sensor_Temperature:MAX31856
Changed lines of the file:
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@@
+	)
+	(symbol
+		(lib_id "Sensor_Temperature:MAX31856")
+		(at 95.25 261.62 0)
+		(unit 1)
+		(exclude_from_sim no)
+		(in_bom yes)
+		(on_board yes)
+		(dnp no)
+		(fields_autoplaced yes)
+		(property "Reference" "U6"
+			(at 99.9841 243.84 0)
+			(effects
+				(font
+					(size 1.27 1.27)
+				)
+				(justify left)
+			)
+		)
+		(property "Value" "MAX31856"
+			(at 99.9841 246.38 0)
+			(effects
+				(font
+					(size 1.27 1.27)
+				)
+				(justify left)
+			)
+		)
+		(property "Footprint" "Package_SO:TSSOP-14_4.4x5mm_P0.65mm"
+			(at 99.06 275.59 0)
+			(effects
+				(font
+					(size 1.27 1.27)
+				)
+				(justify left)
+				(hide yes)
+			)
+		)
+		(property "Datasheet" "https://datasheets.maximintegrated.com/en/ds/MAX31856.pdf"
+			(at 93.98 256.54 0)
+			(effects
+				(font
+					(size 1.27 1.27)
+				)
+				(hide yes)
+			)
+		)
+		(property "Description" "Precision Thermocouple to Digital Converter with Linearization, TSSOP-14"
+			(at 95.25 261.62 0)
+			(effects
+				(font
+					(size 1.27 1.27)
+				)
+				(hide yes)
+			)
+		)
+		(pin "9"
+		)
+		(pin "4"
+		)
+		(pin "13"
+		)
+		(pin "10"
+		)
+		(pin "12"
+		)
+		(pin "1"
+		)
+		(pin "7"
+		)
+		(pin "14"
+		)
+		(pin "6"
+		)
+		(pin "2"
+		)
+		(pin "3"
+		)
+		(pin "11"
+		)
+		(pin "5"
+		)
+		(pin "8"
+		)
+		(instances
+			(project ""
+				(path "/1303051a-0047-4158-8a91-4ef629dc783f"
+					(reference "U6")
+					(unit 1)
+				)
+			)
+		)
 	)
 	(symbol
